File: eagle/smart_watch/board.sch (EAGLE design)
At the start: 7 parts

Commit message: wierd git stuff
Parts:
- removed FRAME1, FRAME2, FRAME3, FRAME4: FRAME-LETTER, SparkFun-Aesthetics:FRAME-LETTER
- added ACCELEROMETER: ADXL345, SparkFun-Sensors:ADXL345
- added C1, C2, C3, C4, C5, C6, C7, C8: (no value), SparkFun-Passives:CAP0402-CAP
- added C10, C11, C12, C13: 0.1uF, SparkFun-Capacitors:.1UF-CER
- added C9: 10uF, SparkFun-Capacitors:10UF-TANT
- added JP2, VIBE: (no value), SparkFun-Connectors:M02-JST-2-PTH-NO_SILK
- added JP3: M05X2PTH, SparkFun-Connectors:M05X2PTH
- added JP4: (no value), SparkFun-Connectors:M04POLAR
- added L1: (no value), SparkFun-Passives:INDUCTOR0402
- added QG1: SM77H, crystal:SM77H
- added R1, R10, R11, R2, R3, R4, R5, R6, R7, R8, R9: (no value), SparkFun-Passives:RESISTOR0402-RES
- added U1: MCP73831, SparkFun-PowerIC:MCP73831
- added U2: TPS61200, SparkFun-PowerIC:TPS61200
- added U3: MAX1704X, SparkFun-PowerIC:MAX1704X
- added U4: V_REG_LDOSMD, SparkFun-PowerIC:V_REG_LDOSMD
Connections:
- new net 3.3V: ACCELEROMETER.VDD, ACCELEROMETER.VSS, C10.1, C11.1, C8.1, C9.+, U$1.VDD1, U$1.VDD2, U3.VDD, U4.OUT
- new net 3.3V_OUT: JP3.10
- new net 5V: C5.1, JP3.2, R8.2, U2.VOUT
- new net 5V_OUT: JP3.1
- new net GND: ACCELEROMETER.GND@2, ACCELEROMETER.GND@4, ACCELEROMETER.GND@5, C1.2, C10.2, C11.2, C12.2, C13.2, C2.2, C4.2, C5.2, C6.2, C7.2, C8.2, C9.-, JP1.GND, JP2.1, JP3.8, JP3.9, QG1.GND, R1.1, R11.2, R2.1, R7.1, R9.1, U1.VSS, U2.GND, U2.PAD@1, U2.PAD@2, U2.PAD@3, U2.PAD@4, U2.PAD@5, U2.PGND, U3.CTG, U3.GND@4, U3.GND@EP, U4.GND, VIBE.1
- new net JTAG_RESETX: JP4.1, U$1.!RESET!/PIO0_0
- new net JTAG_TCLK_SWCLKX: JP4.3, U$1.SWCLK/PIO0_10/SCK0/CT16B0_MAT2
- new net JTAG_TDO_SWOX: JP4.2, U$1.PIO0_9/MOSI0/CT16B0_MAT1
- new net JTAG_TMS_SWDIOX: JP4.4, U$1.SWDIO/PIO1_3/AD4/CT32B1_MAT2
- new net N$1: C13.1, QG1.OUT, U$1.XTALOUT
- new net N$10: R11.1, U3.QST
- new net N$11: C12.1, QG1.VCC, U$1.XTALIN
- new net N$2: R1.2, R2.2, U1.PROG
- new net N$3: C3.2, R3.1, R7.2, U2.UVLO
- new net N$4: C6.1, U2.VAUX
- new net N$5: R6.1, U2.EN
- new net N$6: R5.1, U2.PS
- new net N$7: L1.1, U2.L
- new net N$8: R8.1, R9.2, U2.FB
- new net N$9: C7.1, R10.1, U3.CELL
- new net SCIO1: JP3.6
- new net SCIO2: JP3.4
- new net SCRESET: JP3.7
- new net SCRX: JP3.5
- new net SCTX: JP3.3
- new net VBATT: C1.1, C2.1, C3.1, C4.1, JP1.VCC, JP2.2, L1.2, R3.2, R4.2, R5.2, R6.2, U1.VBAT, U1.VIN, U4.EN, U4.IN
- new net VIBE_PWM: VIBE.2
- new net VIN: R4.1, U2.VIN
Other:
- note added: "3.3V Booster"
- note added: "5V Booster"
- note added: "Battery Connector"
- note added: "Ireg = 1000V/Rprog"
- note added: "Top right corner of screen. Note that wires are mirrored from screen schematic ________ | O| | | |_______|"
- moved on the sheet: JP1, U$1, U$2

Commit message: V1 of Schema is donepending feedback
Parts:
- removed QG1: SM77H, crystal:SM77H
- removed VIBE: (no value), SparkFun-Connectors:M02-JST-2-PTH-NO_SILK
- added LED1, LED2, LED3, LED4: (no value), SparkFun-LED:LED0603
- added R12, R13, R19, R20: Pullup, SparkFun-Passives:RESISTOR0402-RES
- added R14, R16, R17, R18: 330, SparkFun-Passives:RESISTOR0402-RES
- added R15: 10k, SparkFun-Passives:RESISTOR0402-RES
- added S1: (no value), SparkFun-Electromechanical:JOYSTICK_MINI
- added U$3: MOTOR10MM, SparkFun-Electromechanical:MOTOR10MM
- added Y1: (no value), SparkFun-FreqCtrl:CRYSTAL5X3
- C1, C2: value (none) -> 4.7uF
- C12, C13: value 0.1uF -> 16pF; device SparkFun-Capacitors:.1UF-CER -> SparkFun-Passives:CAP0402-CAP
- C3, C6: value (none) -> .1uF
- C4: value (none) -> 10uF
- C5: value (none) -> 22uF
- C7: value (none) -> 1uF
- C8: value (none) -> 10nF
- L1: value (none) -> 4.7uH
- R11: value (none) -> 4.7k
- R2, R5, R6: value (none) -> 10k
- R3, R8: value (none) -> 2M
- R4: value (none) -> 100
- R7, R9: value (none) -> 220k
- U$2: value BLUERADIO_BR-C40NINTERNAL -> BLUETOOTH-RN41"; device SparkFun-RF:BLUERADIO_BR-C40NINTERNAL -> SparkFun-RF:BLUETOOTH-RN41"
Connections:
- new net ACC_INT1: ACCELEROMETER.INT1, U$1.PIO0_2/SSEL0/CT16B0_CAP0
- new net ACC_INT2: ACCELEROMETER.INT2, U$1.PIO0_3
- new net JCENTER: S1.CENT, U$1.PIO3_5
- new net JDOWN: S1.DOWN, U$1.PIO3_2/!DCD!
- new net JLEFT: S1.LEFT, U$1.PIO3_3/!RI!
- new net JRIGHT: S1.RIGHT, U$1.PIO3_4
- new net JUP: S1.UP, U$1.PIO3_1/!DSR!
- new net MISO1: U$1.PIO2_2/!DCD!/MISO1, U$2.SPIMISO
- new net MOSI1: U$1.PIO2_3/!RI!/MOSI1, U$2.SPIMOSI
- new net N$12: LED1.A, U$2.PIO5
- new net N$13: LED1.C, R14.2
- new net N$14: LED2.C, R16.2
- new net N$15: LED3.A, U$1.PIO2_10
- new net N$16: LED4.A, U$1.PIO2_9
- new net N$17: LED3.C, R17.2
- new net N$18: LED4.C, R18.2
- new net SCK1: U$1.PIO2_1/!DSR!/SCK1, U$2.SPICLK
- new net SCL: ACCELEROMETER.SCL, R13.1, R19.1, R20.1, U$1.PIO0_4/SCL, U3.SCL
- new net SDA: ACCELEROMETER.SDA, R12.1, U$1.PIO0_5/SDA, U3.SDA
- new net SSEL1: U$1.PIO2_0/!DTR!/SSEL1, U$2.SPICSB
- new net XTALIN: C13.2, U$1.XTALIN, Y1.2
- new net XTALOUT: C12.2, U$1.XTALOUT, Y1.1
- net 3.3V: now also ACCELEROMETER.CS, R12.2, R13.2, R19.2, R20.2, U$2.VDD
- net GND: now also ACCELEROMETER.SDO, C12.1, C13.1, R14.1, R15.1, R16.1, R17.1, R18.1, S1.GND, U$2.GND, U$2.GND1, U$2.GND2, U$2.GND3, U$2.GND4, U$2.GND5, U$3.-; no longer C12.2, C13.2, QG1.GND, VIBE.1
- net N$1: now also LED2.A, U$2.PIO2; no longer C13.1, QG1.OUT, U$1.XTALOUT
- net N$11: now also R15.2, U$2.PIO4; no longer C12.1, QG1.VCC, U$1.XTALIN
- net SCRX: now also U$1.PIO1_6/RXD/CT32B0_MAT0
- net SCTX: now also U$1.PIO1_7/TXD/CT32B0_MAT1
- net VIBE_PWM: now also U$1.PIO2_5, U$3.+; no longer VIBE.2
Other:
- moved on the sheet: C12, C13

Commit message: Started layout Fixed up joystick wiring
Parts:
- added R21, R22, R23, R24, R25: 10k, SparkFun-Passives:RESISTOR0402-RES
- R10: value (none) -> 1k
- Y1: value (none) -> 16MHz
Connections:
- net 3.3V: now also R21.2, R22.2, R23.2, R24.2, R25.2
- net GND: now also U$1.VSS1, U$1.VSS2
- net JCENTER: now also R25.1, U$1.PIO3_0/!DTR!; no longer U$1.PIO3_5
- net JDOWN: now also R21.1, U$1.R/PIO1_0/AD1/CT32B1_CAP0; no longer U$1.PIO3_2/!DCD!
- net JLEFT: now also R23.1, U$1.R/PIO1_1/AD2/CT32B1_MAT0; no longer U$1.PIO3_3/!RI!
- net JRIGHT: now also R24.1, U$1.R/PIO1_2/AD3/CT32B1_MAT1; no longer U$1.PIO3_4
- net JUP: now also R22.1, U$1.PIO2_11/SCK0; no longer U$1.PIO3_1/!DSR!
- net SCL: no longer R19.1
- net SDA: now also R19.1
Changed lines of the file:
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@@
 <part name="L1" library="SparkFun-Passives" deviceset="INDUCTOR" device="0402" value="4.7uH"/>
 <part name="U3" library="SparkFun-PowerIC" deviceset="MAX1704X" device=""/>
-<part name="R10" library="SparkFun-Passives" deviceset="RESISTOR" device="0402-RES"/>
+<part name="R10" library="SparkFun-Passives" deviceset="RESISTOR" device="0402-RES" value="1k"/>
 <part name="R11" library="SparkFun-Passives" deviceset="RESISTOR" device="0402-RES" value="4.7k"/>
 <part name="C7" library="SparkFun-Passives" deviceset="CAP" device="0402-CAP" value="1uF"/>
@@
 <part name="R12" library="SparkFun-Passives" deviceset="RESISTOR" device="0402-RES" value="Pullup"/>
 <part name="R13" library="SparkFun-Passives" deviceset="RESISTOR" device="0402-RES" value="Pullup"/>
-<part name="Y1" library="SparkFun-FreqCtrl" deviceset="CRYSTAL" device="5X3"/>
+<part name="Y1" library="SparkFun-FreqCtrl" deviceset="CRYSTAL" device="5X3" value="16MHz"/>
 <part name="C12" library="SparkFun-Passives" deviceset="CAP" device="0402-CAP" value="16pF"/>
 <part name="C13" library="SparkFun-Passives" deviceset="CAP" device="0402-CAP" value="16pF"/>
@@
 <part name="R20" library="SparkFun-Passives" deviceset="RESISTOR" device="0402-RES" value="Pullup"/>
 <part name="SUPPLY9" library="SparkFun-Aesthetics" deviceset="3.3V" device=""/>
+<part name="GND35" library="SparkFun-Aesthetics" deviceset="GND" device=""/>
+<part name="R21" library="SparkFun-Passives" deviceset="RESISTOR" device="0402-RES" value="10k"/>
+<part name="R22" library="SparkFun-Passives" deviceset="RESISTOR" device="0402-RES" value="10k"/>
+<part name="R23" library="SparkFun-Passives" deviceset="RESISTOR" device="0402-RES" value="10k"/>
+<part name="R24" library="SparkFun-Passives" deviceset="RESISTOR" device="0402-RES" value="10k"/>
+<part name="R25" library="SparkFun-Passives" deviceset="RESISTOR" device="0402-RES" value="10k"/>
+<part name="SUPPLY10" library="SparkFun-Aesthetics" deviceset="3.3V" device=""/>
 </parts>
 <sheets>
@@
 <instance part="R20" gate="G$1" x="22.86" y="15.24" rot="R90"/>
 <instance part="SUPPLY9" gate="G$1" x="15.24" y="25.4"/>
+<instance part="GND35" gate="1" x="223.52" y="5.08"/>
+<instance part="R21" gate="G$1" x="104.14" y="187.96" rot="R90"/>
+<instance part="R22" gate="G$1" x="111.76" y="187.96" rot="R90"/>
+<instance part="R23" gate="G$1" x="139.7" y="187.96" rot="R90"/>
+<instance part="R24" gate="G$1" x="147.32" y="187.96" rot="R90"/>
+<instance part="R25" gate="G$1" x="154.94" y="187.96" rot="R90"/>
+<instance part="SUPPLY10" gate="G$1" x="127" y="193.04"/>
 </instances>
 <busses>
@@
 <wire x1="114.3" y1="53.34" x2="114.3" y2="50.8" width="0.2032" layer="91"/>
 <pinref part="GND22" gate="1" pin="GND"/>
+</segment>
+<segment>
+<pinref part="U$1" gate="LPC" pin="VSS1"/>
+<wire x1="236.22" y1="17.78" x2="223.52" y2="17.78" width="0.2032" layer="91"/>
+<wire x1="223.52" y1="17.78" x2="223.52" y2="12.7" width="0.2032" layer="91"/>
+<pinref part="U$1" gate="LPC" pin="VSS2"/>
+<wire x1="223.52" y1="12.7" x2="223.52" y2="7.62" width="0.2032" layer="91"/>
+<wire x1="236.22" y1="12.7" x2="223.52" y2="12.7" width="0.2032" layer="91"/>
+<pinref part="GND35" gate="1" pin="GND"/>
 </segment>
 </net>
@@
 <junction x="15.24" y="25.4"/>
 </segment>
+<segment>
+<pinref part="R21" gate="G$1" pin="2"/>
+<pinref part="R22" gate="G$1" pin="2"/>
+<wire x1="104.14" y1="193.04" x2="111.76" y2="193.04" width="0.2032" layer="91"/>
+<pinref part="R23" gate="G$1" pin="2"/>
+<wire x1="139.7" y1="193.04" x2="127" y2="193.04" width="0.2032" layer="91"/>
+<pinref part="R24" gate="G$1" pin="2"/>
+<wire x1="127" y1="193.04" x2="111.76" y2="193.04" width="0.2032" layer="91"/>
+<wire x1="139.7" y1="193.04" x2="147.32" y2="193.04" width="0.2032" layer="91"/>
+<pinref part="R25" gate="G$1" pin="2"/>
+<wire x1="147.32" y1="193.04" x2="154.94" y2="193.04" width="0.2032" layer="91"/>
+<pinref part="SUPPLY10" gate="G$1" pin="3.3V"/>
+<junction x="127" y="193.04"/>
+</segment>
 </net>
 <net name="SCIO2" class="0">
@@
 <segment>
 <pinref part="U3" gate="G$1" pin="SCL"/>
-<wire x1="10.16" y1="2.54" x2="15.24" y2="2.54" width="0.2032" layer="91"/>
 <label x="17.78" y="2.54" size="1.778" layer="95"/>
-<pinref part="R19" gate="G$1" pin="1"/>
-<wire x1="15.24" y1="2.54" x2="22.86" y2="2.54" width="0.2032" layer="91"/>
+<wire x1="10.16" y1="2.54" x2="22.86" y2="2.54" width="0.2032" layer="91"/>
 <wire x1="22.86" y1="2.54" x2="25.4" y2="2.54" width="0.2032" layer="91"/>
-<wire x1="15.24" y1="2.54" x2="15.24" y2="10.16" width="0.2032" layer="91"/>
 <pinref part="R20" gate="G$1" pin="1"/>
 <wire x1="22.86" y1="2.54" x2="22.86" y2="10.16" width="0.2032" layer="91"/>
@@
 <segment>
 <pinref part="U3" gate="G$1" pin="SDA"/>
-<wire x1="10.16" y1="5.08" x2="25.4" y2="5.08" width="0.2032" layer="91"/>
+<wire x1="10.16" y1="5.08" x2="15.24" y2="5.08" width="0.2032" layer="91"/>
 <label x="17.78" y="5.08" size="1.778" layer="95"/>
+<pinref part="R19" gate="G$1" pin="1"/>
+<wire x1="15.24" y1="5.08" x2="25.4" y2="5.08" width="0.2032" layer="91"/>
+<wire x1="15.24" y1="5.08" x2="15.24" y2="10.16" width="0.2032" layer="91"/>
 </segment>
 <segment>
@@
 <wire x1="111.76" y1="175.26" x2="96.52" y2="175.26" width="0.2032" layer="91"/>
 <label x="96.52" y="175.26" size="1.778" layer="95"/>
-</segment>
-<segment>
-<pinref part="U$1" gate="LPC" pin="PIO3_1/!DSR!"/>
-<wire x1="292.1" y1="17.78" x2="307.34" y2="17.78" width="0.2032" layer="91"/>
-<label x="297.18" y="17.78" size="1.778" layer="95"/>
+<pinref part="R22" gate="G$1" pin="1"/>
+<wire x1="111.76" y1="175.26" x2="111.76" y2="182.88" width="0.2032" layer="91"/>
+</segment>
+<segment>
+<wire x1="292.1" y1="25.4" x2="309.88" y2="25.4" width="0.2032" layer="91"/>
+<label x="294.64" y="25.4" size="1.778" layer="95"/>
+<pinref part="U$1" gate="LPC" pin="PIO2_11/SCK0"/>
 </segment>
 </net>
@@
 <segment>
 <pinref part="S1" gate="G$1" pin="DOWN"/>
-<wire x1="111.76" y1="172.72" x2="96.52" y2="172.72" width="0.2032" layer="91"/>
+<wire x1="111.76" y1="172.72" x2="104.14" y2="172.72" width="0.2032" layer="91"/>
 <label x="96.52" y="172.72" size="1.778" layer="95"/>
-</segment>
-<segment>
-<pinref part="U$1" gate="LPC" pin="PIO3_2/!DCD!"/>
-<wire x1="292.1" y1="15.24" x2="307.34" y2="15.24" width="0.2032" layer="91"/>
-<label x="297.18" y="15.24" size="1.778" layer="95"/>
+<pinref part="R21" gate="G$1" pin="1"/>
+<wire x1="104.14" y1="172.72" x2="96.52" y2="172.72" width="0.2032" layer="91"/>
+<wire x1="104.14" y1="172.72" x2="104.14" y2="182.88" width="0.2032" layer="91"/>
+</segment>
+<segment>
+<wire x1="292.1" y1="86.36" x2="309.88" y2="86.36" width="0.2032" layer="91"/>
+<label x="294.64" y="86.36" size="1.778" layer="95"/>
+<pinref part="U$1" gate="LPC" pin="R/PIO1_0/AD1/CT32B1_CAP0"/>
 </segment>
 </net>
@@
 <segment>
 <pinref part="S1" gate="G$1" pin="RIGHT"/>
-<wire x1="137.16" y1="172.72" x2="154.94" y2="172.72" width="0.2032" layer="91"/>
+<wire x1="137.16" y1="172.72" x2="147.32" y2="172.72" width="0.2032" layer="91"/>
 <label x="149.86" y="172.72" size="1.778" layer="95"/>
-</segment>
-<segment>
-<pinref part="U$1" gate="LPC" pin="PIO3_4"/>
-<wire x1="292.1" y1="10.16" x2="307.34" y2="10.16" width="0.2032" layer="91"/>
-<label x="297.18" y="10.16" size="1.778" layer="95"/>
+<pinref part="R24" gate="G$1" pin="1"/>
+<wire x1="147.32" y1="172.72" x2="154.94" y2="172.72" width="0.2032" layer="91"/>
+<wire x1="147.32" y1="172.72" x2="147.32" y2="182.88" width="0.2032" layer="91"/>
+</segment>
+<segment>
+<wire x1="292.1" y1="81.28" x2="309.88" y2="81.28" width="0.2032" layer="91"/>
+<label x="294.64" y="81.28" size="1.778" layer="95"/>
+<pinref part="U$1" gate="LPC" pin="R/PIO1_2/AD3/CT32B1_MAT1"/>
 </segment>
 </net>
@@
 <segment>
 <pinref part="S1" gate="G$1" pin="LEFT"/>
-<wire x1="137.16" y1="175.26" x2="154.94" y2="175.26" width="0.2032" layer="91"/>
+<wire x1="137.16" y1="175.26" x2="139.7" y2="175.26" width="0.2032" layer="91"/>
 <label x="149.86" y="175.26" size="1.778" layer="95"/>
-</segment>
-<segment>
-<pinref part="U$1" gate="LPC" pin="PIO3_3/!RI!"/>
-<wire x1="292.1" y1="12.7" x2="307.34" y2="12.7" width="0.2032" layer="91"/>
-<label x="297.18" y="12.7" size="1.778" layer="95"/>
+<pinref part="R23" gate="G$1" pin="1"/>
+<wire x1="139.7" y1="175.26" x2="154.94" y2="175.26" width="0.2032" layer="91"/>
+<wire x1="139.7" y1="175.26" x2="139.7" y2="182.88" width="0.2032" layer="91"/>
+</segment>
+<segment>
+<wire x1="292.1" y1="83.82" x2="309.88" y2="83.82" width="0.2032" layer="91"/>
+<label x="294.64" y="83.82" size="1.778" layer="95"/>
+<pinref part="U$1" gate="LPC" pin="R/PIO1_1/AD2/CT32B1_MAT0"/>
 </segment>
 </net>
@@
 <wire x1="137.16" y1="170.18" x2="154.94" y2="170.18" width="0.2032" layer="91"/>
 <label x="149.86" y="170.18" size="1.778" layer="95"/>
-</segment>
-<segment>
-<pinref part="U$1" gate="LPC" pin="PIO3_5"/>
-<wire x1="292.1" y1="7.62" x2="307.34" y2="7.62" width="0.2032" layer="91"/>
-<label x="297.18" y="7.62" size="1.778" layer="95"/>
-</segment>
-</net>
+<pinref part="R25" gate="G$1" pin="1"/>
+<wire x1="154.94" y1="170.18" x2="154.94" y2="182.88" width="0.2032" layer="91"/>
+</segment>
+<segment>
+<wire x1="292.1" y1="20.32" x2="309.88" y2="20.32" width="0.2032" layer="91"/>
+<label x="294.64" y="20.32" size="1.778" layer="95"/>
+<pinref part="U$1" gate="LPC" pin="PIO3_0/!DTR!"/>
+</segment>
+</net>
