File: eagle/smart_watch/boardV2.brd (EAGLE design)
At the start: 100 x 80 mm, 49 parts, among them U1 MCP73831, U2 TPS61200, U3 MAX1704X, U4 V_REG_LDOSMD, Y1 16MHz

Commit message: Some updates with git
Parts:
- moved JP4 0.49 mm to (39.6, 1.75)
- moved C5 0.35 mm to (38.5, 34.2)
- moved R9 0.33 mm to (40.0, 34.3)
- moved R3 0.19 mm to (43.1, 34.8)
Routing:
- net 3.3V: track 84.9 -> 83.1 mm
- net ACC_INT2: track 12.7 -> 12.1 mm
