File: eagle/smart_watch/boardV2.sch (EAGLE design)
At the start: 49 parts, among them U1 MCP73831, U2 TPS61200, U3 MAX1704X, U4 V_REG_LDOSMD, Y1 16MHz

Commit message: Some updates with git
Changed lines of the file:
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@@
 <wire x1="218.44" y1="137.16" x2="223.52" y2="137.16" width="0.2032" layer="91"/>
 <pinref part="GND27" gate="1" pin="GND"/>
+<junction x="223.52" y="139.7"/>
+<junction x="223.52" y="142.24"/>
 </segment>
 <segment>
@@
 <segment>
 <pinref part="SUPPLY6" gate="G$1" pin="3.3V"/>
-<pinref part="C10" gate="G$1" pin="1"/>
 <wire x1="218.44" y1="116.84" x2="218.44" y2="111.76" width="0.2032" layer="91"/>
 <pinref part="U$1" gate="LPC" pin="VDD1"/>
-<wire x1="218.44" y1="111.76" x2="218.44" y2="106.68" width="0.2032" layer="91"/>
-<wire x1="218.44" y1="106.68" x2="218.44" y2="101.6" width="0.2032" layer="91"/>
 <wire x1="236.22" y1="111.76" x2="218.44" y2="111.76" width="0.2032" layer="91"/>
+<pinref part="C10" gate="G$1" pin="1"/>
+<wire x1="218.44" y1="111.76" x2="218.44" y2="106.68" width="0.1524" layer="91"/>
+<junction x="218.44" y="111.76"/>
+<pinref part="U$1" gate="LPC" pin="VDD2"/>
+<wire x1="218.44" y1="106.68" x2="218.44" y2="101.6" width="0.1524" layer="91"/>
+<wire x1="228.6" y1="106.68" x2="236.22" y2="106.68" width="0.2032" layer="91"/>
 <pinref part="C11" gate="G$1" pin="1"/>
 <wire x1="228.6" y1="101.6" x2="228.6" y2="106.68" width="0.2032" layer="91"/>
-<pinref part="U$1" gate="LPC" pin="VDD2"/>
-<wire x1="228.6" y1="106.68" x2="236.22" y2="106.68" width="0.2032" layer="91"/>
-<wire x1="228.6" y1="106.68" x2="218.44" y2="106.68" width="0.2032" layer="91"/>
+<wire x1="228.6" y1="106.68" x2="218.44" y2="106.68" width="0.1524" layer="91"/>
+<junction x="228.6" y="106.68"/>
+<junction x="218.44" y="106.68"/>
 </segment>
 <segment>
@@
 </sheet>
 </sheets>
+<errors>
+</errors>
 </schematic>
 </drawing>
