File: eagle/smart_watch/boardV3.sch (EAGLE design)
At the start: 62 parts, among them U1 MCP73831, U2 TPS61200, U3 MAX1704X, U4 V_REG_LDOSMD, Y1 16MHz

Commit message: Did a little of bit of tweeks on the wireing
Parts:
- I2C, RECHARGE: device SparkFun-Connectors:M02POGO_PIN_HOLES_ONLY -> SparkFun-Connectors:M02POLAR
- JP4: device SparkFun-Connectors:M04POLAR -> SparkFun-Connectors:M05PTH
Connections:
- net 3.3V: now also JP4.5
Changed lines of the file:
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@@
 <?xml version="1.0" encoding="utf-8"?>
 <!DOCTYPE eagle SYSTEM "eagle.dtd">
-<eagle version="6.2">
+<eagle version="6.4">
 <drawing>
 <settings>
@@
 <part name="SUPPLY7" library="SparkFun-Aesthetics" deviceset="3.3V" device=""/>
 <part name="GND23" library="SparkFun-Aesthetics" deviceset="GND" device=""/>
-<part name="JP4" library="SparkFun-Connectors" deviceset="M04" device="POLAR"/>
+<part name="JP4" library="SparkFun-Connectors" deviceset="M05" device="PTH"/>
 <part name="C10" library="SparkFun-Passives" deviceset="CAP" device="0603-CAP" value="0.1uF"/>
 <part name="C11" library="SparkFun-Passives" deviceset="CAP" device="0603-CAP" value="0.1uF"/>
@@
 <part name="SUPPLY11" library="SparkFun-Aesthetics" deviceset="3.3V" device=""/>
 <part name="SPI" library="SparkFun-Connectors" deviceset="M04" device="POLAR"/>
-<part name="I2C" library="SparkFun-Connectors" deviceset="M02" device="POGO_PIN_HOLES_ONLY"/>
+<part name="I2C" library="SparkFun-Connectors" deviceset="M02" device="POLAR"/>
 <part name="LED5" library="SparkFun-LED" deviceset="LED" device="0603"/>
 <part name="R23" library="SparkFun-Passives" deviceset="RESISTOR" device="0603-RES" value="330"/>
 <part name="GND39" library="SparkFun-Aesthetics" deviceset="GND" device=""/>
 <part name="SUPPLY12" library="SparkFun-Aesthetics" deviceset="3.3V" device=""/>
-<part name="RECHARGE" library="SparkFun-Connectors" deviceset="M02" device="POGO_PIN_HOLES_ONLY"/>
+<part name="RECHARGE" library="SparkFun-Connectors" deviceset="M02" device="POLAR"/>
 <part name="GND40" library="SparkFun-Aesthetics" deviceset="GND" device=""/>
+<part name="SUPPLY13" library="SparkFun-Aesthetics" deviceset="3.3V" device=""/>
 </parts>
 <sheets>
@@
 <instance part="SUPPLY7" gate="G$1" x="114.3" y="116.84"/>
 <instance part="GND23" gate="1" x="111.76" y="76.2"/>
-<instance part="JP4" gate="G$1" x="327.66" y="129.54" rot="MR0"/>
+<instance part="JP4" gate="G$1" x="335.28" y="132.08" rot="MR0"/>
 <instance part="C10" gate="G$1" x="218.44" y="96.52"/>
 <instance part="C11" gate="G$1" x="228.6" y="96.52"/>
@@
 <instance part="RECHARGE" gate="G$1" x="170.18" y="50.8" rot="R180"/>
 <instance part="GND40" gate="1" x="149.86" y="35.56"/>
+<instance part="SUPPLY13" gate="G$1" x="307.34" y="142.24" rot="MR0"/>
 </instances>
 <busses>
@@
 <pinref part="SUPPLY12" gate="G$1" pin="3.3V"/>
 </segment>
+<segment>
+<pinref part="JP4" gate="G$1" pin="5"/>
+<wire x1="327.66" y1="137.16" x2="322.58" y2="137.16" width="0.2032" layer="91"/>
+<wire x1="322.58" y1="137.16" x2="307.34" y2="137.16" width="0.1524" layer="91"/>
+<wire x1="307.34" y1="137.16" x2="307.34" y2="142.24" width="0.1524" layer="91"/>
+<pinref part="SUPPLY13" gate="G$1" pin="3.3V"/>
+</segment>
 </net>
 <net name="SCIO2" class="0">
@@
 <segment>
 <pinref part="JP4" gate="G$1" pin="4"/>
-<wire x1="322.58" y1="134.62" x2="309.88" y2="134.62" width="0.2032" layer="91"/>
+<wire x1="327.66" y1="134.62" x2="309.88" y2="134.62" width="0.2032" layer="91"/>
 <label x="299.72" y="134.62" size="1.778" layer="95"/>
 </segment>
@@
 <segment>
 <pinref part="JP4" gate="G$1" pin="3"/>
-<wire x1="322.58" y1="132.08" x2="309.88" y2="132.08" width="0.2032" layer="91"/>
+<wire x1="327.66" y1="132.08" x2="309.88" y2="132.08" width="0.2032" layer="91"/>
 <label x="299.72" y="132.08" size="1.778" layer="95"/>
 </segment>
@@
 <segment>
 <pinref part="JP4" gate="G$1" pin="2"/>
-<wire x1="322.58" y1="129.54" x2="309.88" y2="129.54" width="0.2032" layer="91"/>
+<wire x1="327.66" y1="129.54" x2="309.88" y2="129.54" width="0.2032" layer="91"/>
 <label x="299.72" y="129.54" size="1.778" layer="95"/>
 </segment>
@@
 <segment>
 <pinref part="JP4" gate="G$1" pin="1"/>
-<wire x1="322.58" y1="127" x2="309.88" y2="127" width="0.2032" layer="91"/>
+<wire x1="327.66" y1="127" x2="309.88" y2="127" width="0.2032" layer="91"/>
 <label x="299.72" y="127" size="1.778" layer="95"/>
 </segment>

Commit message: Fixed up git ignore for xpress;
Parts:
- JP2: device SparkFun-Connectors:M02-JST-2-PTH-NO_SILK -> SparkFun-Connectors:M02PTH
Changed lines of the file:
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@@
 <part name="U$1" library="lpc1100v1.1" deviceset="LPC1113/14-LQFP48" device=""/>
 <part name="U1" library="SparkFun-PowerIC" deviceset="MCP73831" device=""/>
-<part name="JP2" library="SparkFun-Connectors" deviceset="M02" device="-JST-2-PTH-NO_SILK"/>
+<part name="JP2" library="SparkFun-Connectors" deviceset="M02" device="PTH"/>
 <part name="C1" library="SparkFun-Passives" deviceset="CAP" device="0603-CAP" value="4.7uF"/>
 <part name="GND2" library="SparkFun-Aesthetics" deviceset="GND" device=""/>
