File: eagle/smart_watch/boardV4.brd (EAGLE design)
At the start: 63.6 x 36.1 mm, 67 parts, among them IC1 SC16IS750, U1 MCP73831, U2 TPS61200, U3 MAX1704X, U4 V_REG_LDOSMD, Y1 16MHz, Y2 12.28MHz

Commit message: Some more tweaks
Parts:
- moved C13 4.04 mm to (23.6, 1.61), turned to 180 degrees
- moved R15 2.84 mm to (9.27, 21.0), turned to 90 degrees
- moved I2C 2.41 mm to (13.3, 10.5), turned to 0 degrees
- moved U$4 1.88 mm to (10.8, 8.00)
- moved U3 1.71 mm to (22.3, 20.1)
- moved R11 1.31 mm to (22.7, 16.5)
- moved C12 0.97 mm to (28.7, 4.33)
- moved C1 0.64 mm to (5.42, 29.2)
- moved JP4 0.46 mm to (30.0, 1.60)
- moved JP2 0.40 mm to (12.1, 34.3)
- moved IC1 0.40 mm to (4.70, 21.5)
- moved ACCELEROMETER 0.13 mm to (23.8, 11.9)
Routing:
- added copper zone on layer 1, net GND
- added copper zone on layer 16, net GND

Commit message: Did a bunch of routing, woo... woo!!! woo?
Parts:
- moved C2 20.9 mm to (14.6, 27.2), turned to 180 degrees
- moved R14 19.7 mm to (8.89, 21.7)
- moved R24 18.7 mm to (2.92, 18.4)
- moved R26 17.7 mm to (2.79, 20.3), turned to 0 degrees
- moved C10 11.9 mm to (23.0, 9.11), turned to 90 degrees
- moved R25 11.8 mm to (2.92, 16.6), turned to 0 degrees
- moved C11 11.6 mm to (33.4, 17.3), turned to 0 degrees
- moved LED6 11.5 mm to (6.73, 18.4), turned to 90 degrees
- moved RECHARGE 10.9 mm to (2.67, 23.6), turned to 90 degrees
- moved C16 10.4 mm to (7.75, 24.1), turned to 270 degrees
- moved LED7 9.04 mm to (6.73, 20.3), turned to 90 degrees
- moved IC1 7.75 mm to (12.1, 19.1), turned to 270 degrees
- moved R13 7.62 mm to (21.6, 17.9), turned to 0 degrees
- moved R15 7.51 mm to (16.8, 21.5), turned to 0 degrees
- moved C17 6.67 mm to (15.6, 24.3)
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Routing:
- net 3.3V: track 0.00 -> 114.6 mm, vias 0 -> 6
- net SDA: track 0.00 -> 65.6 mm, vias 0 -> 3
- net SCL: track 0.00 -> 60.8 mm, vias 0 -> 2
- net GND: track 0.00 -> 52.5 mm, vias 0 -> 4
- net JRIGHT: track 0.00 -> 37.5 mm
- net JDOWN: track 0.00 -> 32.2 mm
- net JUP: track 0.00 -> 23.8 mm
- net JLEFT: track 0.00 -> 23.8 mm
- net JCENTER: track 0.00 -> 22.9 mm
- net SCRX: track 0.00 -> 21.1 mm, vias 0 -> 1
- net SCTX: track 0.00 -> 15.4 mm, vias 0 -> 1
- net JTAG_TMS_SWDIOX: track 0.00 -> 13.6 mm, vias 0 -> 1
- net XTALIN: track 0.00 -> 12.7 mm
- net JTAG_RESETX: track 0.00 -> 11.5 mm
- net JTAG_TDO_SWOX: track 0.00 -> 11.2 mm
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
Commit message: version 4.0 all connected
Parts:
- moved C5 10.4 mm to (27.1, 24.8)
- moved R5 10.0 mm to (21.3, 28.6)
- moved U4 7.87 mm to (27.4, 21.1), turned to 180.4 degrees
- moved R8 7.78 mm to (27.1, 26.2)
- moved C4 6.56 mm to (33.0, 24.2)
- moved C15 6.38 mm to (33.0, 22.8)
- moved C2 3.61 mm to (11.0, 27.8), turned to 270 degrees
- moved C7 3.01 mm to (25.2, 22.2)
- moved R9 1.92 mm to (29.4, 25.4), turned to 90 degrees
- moved R11 1.78 mm to (19.5, 20.0)
- moved C14 1.67 mm to (36.8, 20.0)
- moved R10 1.12 mm to (22.2, 25.8), turned to 0 degrees
- moved U2 1.08 mm to (19.9, 31.7)
- moved R7 0.90 mm to (16.8, 30.3), turned to 270.3 degrees
- moved U3 0.85 mm to (22.8, 21.7)
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Routing:
- net 3.3V: track 114.6 -> 159.9 mm, vias 6 -> 9
- net VBATT: track 11.1 -> 45.2 mm, vias 0 -> 2
- net GND: track 52.5 -> 75.3 mm, vias 4 -> 6
- net 5V: track 0.00 -> 15.9 mm, vias 0 -> 2
- net N$8: track 0.00 -> 11.2 mm
- net N$5: track 0.00 -> 9.20 mm, vias 0 -> 2
- net VIN: track 0.39 -> 8.87 mm
- net N$3: track 0.00 -> 8.09 mm
- net N$9: track 0.00 -> 6.92 mm
- net N$7: track 0.00 -> 4.76 mm
- net N$10: track 0.00 -> 2.89 mm
- net N$4: track 0.00 -> 2.28 mm
- net SCL: track 60.8 -> 62.9 mm
- net N$6: track 0.00 -> 1.81 mm
- net N$1: track 8.88 -> 10.1 mm
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